File: hw/v2.3/main-board/pmic.kicad_sch (KiCad schematic)
At the start: 25 parts, among them J3 USB_C_Receptacle, J4 Conn_01x03_MountingPin, Q1 AP3400, Q2 AP3401, U2 UAT56A05L05, U3 MCP73832, U4 TLV62569DRL

Commit message: Update r2.3
- Add make panel KiKit script
- Add production gerbers
Parts:
- R10: Mfg Yageo -> (none); PN AC0402FR-0747KL -> (none)
- R9: Mfg Yageo -> (none); PN AC0402FR-07210KL -> (none)
Changed lines of the file:
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@@
       (effects (font (size 1.27 1.27)) hide)
     )
-    (property "PN" "AC0402FR-07210KL" (id 4) (at 200.66 133.35 0)
+    (property "PN" "" (id 4) (at 200.66 133.35 0)
       (effects (font (size 1.27 1.27)) hide)
     )
-    (property "Mfg" "Yageo" (id 5) (at 200.66 133.35 0)
+    (property "Mfg" "" (id 5) (at 200.66 133.35 0)
       (effects (font (size 1.27 1.27)) hide)
     )
@@
       (effects (font (size 1.27 1.27)) hide)
     )
-    (property "PN" "AC0402FR-0747KL" (id 4) (at 200.66 146.05 0)
+    (property "PN" "" (id 4) (at 200.66 146.05 0)
       (effects (font (size 1.27 1.27)) hide)
     )
-    (property "Mfg" "Yageo" (id 5) (at 200.66 146.05 0)
+    (property "Mfg" "" (id 5) (at 200.66 146.05 0)
       (effects (font (size 1.27 1.27)) hide)
     )
